File: schematic/MT3608_1.kicad_sch (KiCad schematic)
At the start: 9 parts, among them IC3 TPS630250RNCR

Commit message: Routing
Parts:
- IC3: footprint TPS630250RNCR -> TPS630250RNCR:TPS630250RNCR
- L2: footprint MACHADA_footprints:CYA1040-22UH -> Inductor_SMD:L_Chilisin_BMRx00050512-B; MPN CYA1040-22UH -> YSPI0530S-1R0M
Connections:
- net power_input: now also IC3.10 (PFM/PWM), IC3.8 (EN)
Changed lines of the file:
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@@
+	)
+	(junction
+		(at 106.68 129.54)
+		(diameter 0)
+		(color 0 0 0 0)
 	)
 	(junction
@@
 	(wire
 		(pts
+			(xy 106.68 86.36) (xy 106.68 129.54)
+		)
+		(stroke
+			(width 0)
+			(type default)
+		)
+	)
+	(wire
+		(pts
 			(xy 224.79 125.73) (xy 238.76 125.73)
 		)
@@
 	(wire
 		(pts
-			(xy 90.17 129.54) (xy 139.7 129.54)
+			(xy 90.17 129.54) (xy 106.68 129.54)
 		)
 		(stroke
@@
 	(wire
 		(pts
-			(xy 106.68 129.54) (xy 106.68 86.36)
-		)
-		(stroke
-			(width 0)
-			(type default)
-		)
-	)
-	(wire
-		(pts
 			(xy 172.72 115.57) (xy 182.88 115.57)
 		)
@@
 		(pts
 			(xy 177.8 123.19) (xy 177.8 124.46)
+		)
+		(stroke
+			(width 0)
+			(type default)
+		)
+	)
+	(wire
+		(pts
+			(xy 106.68 129.54) (xy 139.7 129.54)
 		)
 		(stroke
@@
 			)
 		)
-		(property "Footprint" "TPS630250RNCR"
+		(property "Footprint" "TPS630250RNCR:TPS630250RNCR"
 			(at 168.91 210.49 0)
 			(effects
@@
 			)
 		)
-		(property "Footprint" "MACHADA_footprints:CYA1040-22UH"
+		(property "Footprint" "Inductor_SMD:L_Chilisin_BMRx00050512-B"
 			(at 130.81 110.49 0)
 			(effects
@@
 			)
 		)
-		(property "MPN" "CYA1040-22UH"
+		(property "MPN" "YSPI0530S-1R0M"
 			(at 130.81 111.76 90)
 			(effects
