File: schematic/MT3608_5V_BOOST_CONVERTOR.kicad_sch (KiCad schematic)
At the start: 13 parts, among them U2 MT3608

Commit message: Routing
Parts:
- L1: footprint MACHADA_footprints:CYA1040-22UH -> Inductor_SMD:L_Chilisin_BMRG00101030
Changed lines of the file:
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@@
+		)
+	)
+	(label "5v"
+		(at 207.01 88.9 0)
+		(effects
+			(font
+				(size 1.27 1.27)
+			)
+			(justify left bottom)
 		)
 	)
@@
 		(pin "1"
 		)
+		(instances
+			(project "schematic"
+				(path "/374f5031-bd65-4a4b-92ce-befdd0c9f08b/f360cbf4-248e-49bd-9da6-3bb057d11a5f"
+					(reference "C8")
+					(unit 1)
+				)
+			)
+		)
 	)
 	(symbol
@@
 		(dnp no)
 		(fields_autoplaced yes)
-		(property "Reference" "#PWR017"
+		(property "Reference" "#PWR0102"
 			(at 193.04 102.87 0)
 			(effects
@@
 		)
 		(pin "1"
+		)
+		(instances
+			(project "schematic"
+				(path "/374f5031-bd65-4a4b-92ce-befdd0c9f08b/f360cbf4-248e-49bd-9da6-3bb057d11a5f"
+					(reference "#PWR0102")
+					(unit 1)
+				)
+			)
 		)
 	)
@@
 		(dnp no)
 		(fields_autoplaced yes)
-		(property "Reference" "#PWR09"
+		(property "Reference" "#PWR0101"
 			(at 105.41 116.84 0)
 			(effects
@@
 		)
 		(pin "1"
+		)
+		(instances
+			(project "schematic"
+				(path "/374f5031-bd65-4a4b-92ce-befdd0c9f08b/f360cbf4-248e-49bd-9da6-3bb057d11a5f"
+					(reference "#PWR0101")
+					(unit 1)
+				)
+			)
 		)
 	)
@@
 		(pin "1"
 		)
+		(instances
+			(project "schematic"
+				(path "/374f5031-bd65-4a4b-92ce-befdd0c9f08b/f360cbf4-248e-49bd-9da6-3bb057d11a5f"
+					(reference "C7")
+					(unit 1)
+				)
+			)
+		)
 	)
 	(symbol
@@
 		)
 		(pin "2"
+		)
+		(instances
+			(project "schematic"
+				(path "/374f5031-bd65-4a4b-92ce-befdd0c9f08b/f360cbf4-248e-49bd-9da6-3bb057d11a5f"
+					(reference "R3")
+					(unit 1)
+				)
+			)
 		)
 	)
@@
 		(pin "2"
 		)
+		(instances
+			(project "schematic"
+				(path "/374f5031-bd65-4a4b-92ce-befdd0c9f08b/f360cbf4-248e-49bd-9da6-3bb057d11a5f"
+					(reference "D1")
+					(unit 1)
+				)
+			)
+		)
 	)
 	(symbol
@@
 		(pin "2"
 		)
+		(instances
+			(project "schematic"
+				(path "/374f5031-bd65-4a4b-92ce-befdd0c9f08b/f360cbf4-248e-49bd-9da6-3bb057d11a5f"
+					(reference "R2")
+					(unit 1)
+				)
+			)
+		)
 	)
 	(symbol
@@
 		)
 		(pin "2"
+		)
+		(instances
+			(project "schematic"
+				(path "/374f5031-bd65-4a4b-92ce-befdd0c9f08b/f360cbf4-248e-49bd-9da6-3bb057d11a5f"
+					(reference "R1")
+					(unit 1)
+				)
+			)
 		)
 	)
@@
 		(pin "1"
 		)
+		(instances
+			(project "schematic"
+				(path "/374f5031-bd65-4a4b-92ce-befdd0c9f08b/f360cbf4-248e-49bd-9da6-3bb057d11a5f"
+					(reference "C2")
+					(unit 1)
+				)
+			)
+		)
 	)
 	(symbol
@@
 		(dnp no)
 		(fields_autoplaced yes)
-		(property "Reference" "#PWR016"
+		(property "Reference" "#PWR0103"
 			(at 176.53 123.19 0)
 			(effects
@@
 		(pin "1"
 		)
+		(instances
+			(project "schematic"
+				(path "/374f5031-bd65-4a4b-92ce-befdd0c9f08b/f360cbf4-248e-49bd-9da6-3bb057d11a5f"
+					(reference "#PWR0103")
+					(unit 1)
+				)
+			)
+		)
 	)
 	(symbol
@@
 			)
 		)
-		(property "Footprint" "MACHADA_footprints:CYA1040-22UH"
+		(property "Footprint" "Inductor_SMD:L_Chilisin_BMRG00101030"
 			(at 149.86 88.9 0)
 			(effects
@@
 		(pin "2"
 		)
+		(instances
+			(project "schematic"
+				(path "/374f5031-bd65-4a4b-92ce-befdd0c9f08b/f360cbf4-248e-49bd-9da6-3bb057d11a5f"
+					(reference "L1")
+					(unit 1)
+				)
+			)
+		)
 	)
 	(symbol
@@
 		(dnp no)
 		(fields_autoplaced yes)
-		(property "Reference" "#PWR010"
+		(property "Reference" "#PWR0104"
 			(at 149.86 118.11 0)
 			(effects
@@
 		)
 		(pin "1"
+		)
+		(instances
+			(project "schematic"
+				(path "/374f5031-bd65-4a4b-92ce-befdd0c9f08b/f360cbf4-248e-49bd-9da6-3bb057d11a5f"
+					(reference "#PWR0104")
+					(unit 1)
+				)
+			)
 		)
 	)
@@
 		(pin "1"
 		)
+		(instances
+			(project "schematic"
+				(path "/374f5031-bd65-4a4b-92ce-befdd0c9f08b/f360cbf4-248e-49bd-9da6-3bb057d11a5f"
+					(reference "C1")
+					(unit 1)
+				)
+			)
+		)
 	)
 	(symbol
@@
 		(pin "1"
 		)
+		(instances
+			(project "schematic"
+				(path "/374f5031-bd65-4a4b-92ce-befdd0c9f08b/f360cbf4-248e-49bd-9da6-3bb057d11a5f"
+					(reference "C3")
+					(unit 1)
+				)
+			)
+		)
 	)
 	(symbol
@@
 		(pin "6"
 		)
+		(instances
+			(project "schematic"
+				(path "/374f5031-bd65-4a4b-92ce-befdd0c9f08b/f360cbf4-248e-49bd-9da6-3bb057d11a5f"
+					(reference "U2")
+					(unit 1)
+				)
+			)
+		)
 	)
 	(symbol
@@
 		(pin "1"
 		)
+		(instances
+			(project "schematic"
+				(path "/374f5031-bd65-4a4b-92ce-befdd0c9f08b/f360cbf4-248e-49bd-9da6-3bb057d11a5f"
+					(reference "C9")
+					(unit 1)
+				)
+			)
+		)
 	)
 	(symbol
@@
 		(pin "1"
 		)
-	)
+		(instances
+			(project "schematic"
+				(path "/374f5031-bd65-4a4b-92ce-befdd0c9f08b/f360cbf4-248e-49bd-9da6-3bb057d11a5f"
+					(reference "TP1")
+					(unit 1)
+				)
+			)
+		)
+	)
