File: schematic/_autosave-SIM808_GPRS_GPSS_MODULE.kicad_sch (KiCad schematic)
At the start: 37 parts, among them IC4 SIM7600G-H_R2, J10 SIM_Card_Shielded, Q1 BC817, Q15 SI2302, Q16 SI2302, Q2 BC817

Commit message: Routing
Parts:
- removed J10: SIM_Card_Shielded, Connector_JAE:JAE_SIM_Card_SF72S006, symbol fridgeduino-rescue:SIM_Card_Shielded-Connector-gsm_lora_logger-rescue-gsm_lora_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
- added J1: SIM7155-6-1-14-A, SIM7155-6-1-14-A_GCT, symbol simHolderPush:SIM7155-6-1-14-A
- AE3, AE4: footprint greencharge-footprints:UFL_COAX_CONN23370191 -> antenna:CONN_2337019-1_TEC
Connections:
- net GND: now also J1.C5 (GND), J1.CD, J1.GND1, J1.GND2, J1.GND3, J1.GND4, J1.GND5, J1.GND6
- net SIM_DATA: now also J1.C7 (I/O)
- net SIM_VDD: now also J1.C1 (VCC)
- net at D25.3 (TVS2), R88.1: now also J1.C2 (RST)
- net at D25.4 (TVS3), R89.1: now also J1.C3 (CLK)
Other:
- moved on the sheet: C74, C75, D25, D26, D27, Q1, Q15, Q16, Q2, R87, R88, R89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
