File: schematic/schematic.kicad_sch (KiCad schematic)
At the start: 1 part, among them U1 ESP32-S3-WROOM-1

Commit message: Second
Parts:
- added IC1: SIM7080G, SIM7080G, symbol SIM7080G:SIM7080G
- added IC2: AXP2101, QFN40P500X500X80-41N-D, symbol axp2101:AXP2101
- added J1: Micro_SD_Card_Det2, symbol Connector:Micro_SD_Card_Det2
- added J2: SIM_Card, symbol Connector:SIM_Card

Commit message: shcematic complete
Parts:
- removed IC2: AXP2101, QFN40P500X500X80-41N-D, symbol axp2101:AXP2101
- removed J1: Micro_SD_Card_Det2, symbol Connector:Micro_SD_Card_Det2
- removed J2: SIM_Card, symbol Connector:SIM_Card
- added C25, C28: 4.7u, Capacitor_SMD:C_0402_1005Metric_Pad0.74x0.62mm_HandSolder, symbol Device:C_Small
- added C26: 10n, Capacitor_SMD:C_0402_1005Metric_Pad0.74x0.62mm_HandSolder, symbol Device:C_Small
- added C27, C29, C32: 100n, Capacitor_SMD:C_0402_1005Metric_Pad0.74x0.62mm_HandSolder, symbol Device:C_Small
- added C4: 10u, Capacitor_SMD:C_0402_1005Metric, symbol Device:C_Small
- added C5, C6: 0.1u, Capacitor_SMD:C_0402_1005Metric, symbol Device:C_Small
- added D15, D16: SP0502BAHT, Package_TO_SOT_SMD:SOT-23, symbol Power_Protection:SP0502BAHT
- added D23: PWR, LED_SMD:LED_0603_1608Metric, symbol Device:LED_Small
- added IC?: AS312, AS312, symbol AS312:AS312
- added J3: USB_C_Receptacle_USB2.0, greencharge-footprints:MC-311D_USB_C_2.0_12PIN, symbol Connector:USB_C_Receptacle_USB2.0
- added L3: 2A_bead, Inductor_SMD:L_0603_1608Metric, symbol Device:L_Ferrite
- added R12: 10k, Resistor_SMD:R_0402_1005Metric, symbol fridgeduino-rescue:R_Small_US-Device
- added R13: 10k, Resistor_SMD:R_0402_1005Metric, symbol Device:R_Small_US
- added R14: 4.7k, Resistor_SMD:R_0402_1005Metric, symbol fridgeduino-rescue:R_Small_US-Device
- added R15: 1k, Resistor_SMD:R_0402_1005Metric, symbol fridgeduino-rescue:R_Small_US-Device
- added R31, R81: 5.1K, Resistor_SMD:R_0402_1005Metric, symbol Device:R_US
- added R32: 1K, Resistor_SMD:R_0402_1005Metric, symbol Device:R_US
- added R76: 1K, Resistor_SMD:R_0402_1005Metric, symbol Device:R_Small
- added SW2, SW3: SW_Push, greencharge-footprints:SKRPACE010, symbol Switch:SW_Push
- added U?: AM2302, Sensor:ASAIR_AM2302_P2.54mm_Vertical, symbol Sensor:AM2302
- added Z1: MMSZ5231B-7-F, digikey-footprints:SOD-123, symbol dk_Diodes-Zener-Single:MMSZ5231B-7-F
Connections:
- net at IC1.34 (VBAT_1): now also IC1.35 (VBAT_2)
- net LED2: now reaches IC1.42 (STATUS)
- net GND: now reaches IC1.69 (GND_15)
- net GND: now also IC1.70 (GND_16), IC1.71 (GND_17), IC1.72 (GND_18), IC1.73 (GND_19), IC1.74 (GND_20), IC1.75 (GND_21), IC1.76 (GND_22), IC1.77 (GND_23), U1.1 (GND), U1.40 (GND), U1.41 (GND), C25.2, C26.2, C27.2, C28.2, C29.1, C32.1, C4.2, C5.2, C6.2, D15.3 (A), D16.3 (A), D23.1 (K), IC?.3 (VSS), J3.A1 (GND), J3.A12 (GND), J3.B1 (GND), J3.B12 (GND), J3.S1 (SHIELD), R31.2, R32.2, R81.2, SW2.1, SW3.1, U?.3 (GND), U?.4 (GND)
- net ESP_TX: now reaches U1.10 (IO17)
- net ESP_RX: now reaches U1.11 (IO18)
- net D-: now reaches U1.13 (USB_D-)
- net D-: now also D15.1 (K), J3.A7 (D-), J3.B7 (D-)
- net D+: now reaches U1.14 (USB_D+)
- net D+: now also D15.2 (K), J3.A6 (D+), J3.B6 (D+)
- net +3V3: now reaches U1.2 (3V3)
- net +3V3: now also C29.2, C32.2, C4.1, C5.1, IC?.1 (VDD), R12.1, R13.1, R14.1, R76.1, U?.1 (VDD)
- net DHT22_Data: now reaches U1.22 (IO14)
- net DHT22_Data: now also R14.2, U?.2 (SDA)
- net boot: now reaches U1.27 (IO0)
- net boot: now also R13.2, SW3.2
- net ~{esp_rst}: now reaches U1.3 (EN)
- net ~{esp_rst}: now also C6.1, R12.2, SW2.2
- net Motion_out: now reaches U1.8 (IO15)
- net Motion_out: now also R15.1
- new net: D23.2 (A), R76.2
- new net: D16.1 (K), J3.B5 (CC2), R31.1
- new net: IC?.2 (REL), R15.2
- new net: R32.1, Z1.A
- new net: D16.2 (K), J3.A5 (CC1), R81.1
- new net +5V: C27.1, C28.1, L3.1
- new net VBUS: C25.1, C26.1, J3.A4 (VBUS), J3.A9 (VBUS), J3.B4 (VBUS), J3.B9 (VBUS), L3.2, Z1.K
- no-connect marks 0 -> 4
Other:
- added sheet BUCK_CONVERTER_3V3_2A_TPS56339DDCR (BUCK_CONVERTER_3V3_2A_TPS56339DDCR.kicad_sch)
- added sheet LIPO_BAT_CHARGER_TP4056 (LIPO_BAT_CHARGER_TP4056.kicad_sch)
- added sheet MT3608_1.2mHz_STEP-UP_CONVERTOR (MT3608_1.kicad_sch)
- added sheet MT3608_5V_BOOST_CONVERTOR (MT3608_5V_BOOST_CONVERTOR.kicad_sch)
- added sheet POWER_PATH_SELECTOR (POWER_PATH_SELECTOR.kicad_sch)
- added sheet SIM808_GPRS_GPS_MODULE (SIM808_GPRS_GPSS_MODULE.kicad_sch)
- note added: "Micro USB Interface"
- moved on the sheet: IC1, U1

Commit message: Routing
Parts:
- removed IC1: SIM7080G, SIM7080G, symbol SIM7080G:SIM7080G
- removed R32: 1K, Resistor_SMD:R_0402_1005Metric, symbol Device:R_US
- removed Z1: MMSZ5231B-7-F, digikey-footprints:SOD-123, symbol dk_Diodes-Zener-Single:MMSZ5231B-7-F
- IC2: renamed from IC?; footprint AS312 -> as312:AS312
- J3: footprint greencharge-footprints:MC-311D_USB_C_2.0_12PIN -> Connector_USB:USB_C_Receptacle_GCT_USB4105-xx-A_16P_TopMnt_Horizontal
- SW2, SW3: footprint greencharge-footprints:SKRPACE010 -> button:SMT_4.2X3.2_
- gave numbers to parts that had none: 1
Connections:
- no-connect marks 4 -> 2
Other:
- moved on the sheet: C29, C32, C4, C5, C6, D23, IC2, R12, R13, R14, R15, R76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
