File: schematic/schematic.kicad_pcb (KiCad board)
At the start: 2 copper layers, 93.8 x 81.6 mm, 114 parts, among them IC2 AS312, IC3 TPS630250RNCR, IC4 SIM7600G-H_R2, J10 SIM_Card_Shielded, J3 USB_C_Receptacle_USB2.0, Q1 BC817, Q15 SI2302, Q16 SI2302, Q2 BC817, Q8 NCE6005AR, Q9 NCE6005AR, U1 ESP32-S3-WROOM-1, U10 TPS56339DDC, U2 MT3608, U3 AM2302

Commit message: Routing
Parts:
- removed J10: SIM_Card_Shielded, Connector_JAE:JAE_SIM_Card_SF72S006
- removed R32: 1K, Resistor_SMD:R_0402_1005Metric
- added AE3: GPRS_ANTENNA, antenna:CONN_2337019-1_TEC, B.Cu at (145.1, 125.1)
- added AE4: GPS_ANTENNA, antenna:CONN_2337019-1_TEC, B.Cu at (104.1, 83.1)
- added J1: SIM7155-6-1-14-A, simHolderpush:SIM7155-6-1-14-A_GCT, F.Cu at (106.8, 115.0)
- added J9: BATT_CONNECTOR, TerminalBlock_Phoenix:TerminalBlock_Phoenix_PTSM-0,5-2-HV-2.5-SMD_1x02-1MP_P2.50mm_Vertical, F.Cu at (150.1, 122.3)
- added L1: 22uH, Inductor_SMD:L_Chilisin_BMRG00101030, F.Cu at (161.3, 63.6)
- added L2: 1uH, Inductor_SMD:L_Chilisin_BMRx00050512-B, F.Cu at (140.8, 78.0)
- added L5: 4.7uH, Inductor_SMD:L_Chilisin_BMRx00050512-B, F.Cu at (155.1, 85.5)
- added SW2: SW_Push, button:SMT_4.2X3.2_, F.Cu at (119.5, 60.6)
- added SW3: SW_Push, button:SMT_4.2X3.2_, F.Cu at (150.6, 65.5)
- added U4: TP4056, tp4056:SOIC127P600X175-9N, F.Cu at (145.6, 103.5)
- C23, C66, C67, C68, C70, C71, IC4, L9, R82, R86: moved to B.Cu
- moved R97 80.5 mm to (106.2, 89.7)
- moved C28 78.8 mm to (120.0, 54.3), turned to -90 degrees
- moved D26 78.7 mm to (108.7, 96.4), turned to 180 degrees
- moved C26 78.5 mm to (118.1, 52.4), turned to -90 degrees
- moved C25 78.2 mm to (116.2, 52.3), turned to -90 degrees
- moved C68 77.8 mm to (100.7, 116.8), turned to 90 degrees
- moved R93 77.2 mm to (106.2, 100.2)
- moved R95 76.8 mm to (106.6, 103.1), turned to 90 degrees
- moved C66 76.8 mm to (102.0, 116.9), turned to 90 degrees
- moved U3 76.8 mm to (166.4, 123.4)
- moved C27 76.5 mm to (121.4, 54.2), turned to -90 degrees
- moved C70 76.2 mm to (104.3, 88.2), turned to 90 degrees
- moved R98 76.1 mm to (111.9, 83.4), turned to 90 degrees
- moved R87 75.2 mm to (104.2, 85.0)
- moved R99 73.5 mm to (114.1, 87.4), turned to 90 degrees
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Connections:
- net /BUCK_CONVERTER_3V3_2A_TPS56339DDCR/pwr_IN renamed /MT3608_5V_BOOST_CONVERTOR/5v
- C59 pad 1: /LIPO_BAT_CHARGER_TP4056/POWER_NPUT -> +5V
- C60 pad 1: /LIPO_BAT_CHARGER_TP4056/POWER_NPUT -> +5V
- C61 pad 1: /LIPO_BAT_CHARGER_TP4056/POWER_NPUT -> +5V
- C62 pad 1: /LIPO_BAT_CHARGER_TP4056/POWER_NPUT -> +5V
- D17 pad 2: VBUS -> +5V
- IC3 pad 10: Net-(IC3-EN) -> /MT3608_1.2mHz_STEP-UP_CONVERTOR/power_input
- IC3 pad 8: Net-(IC3-EN) -> /MT3608_1.2mHz_STEP-UP_CONVERTOR/power_input
- R24 pad 1: VBUS -> +5V
- R77 pad 1: /LIPO_BAT_CHARGER_TP4056/POWER_NPUT -> +5V
- R78 pad 1: /LIPO_BAT_CHARGER_TP4056/POWER_NPUT -> +5V
Routing:
- net GND: track 0.00 -> 344.2 mm, vias 0 -> 232
- net 4.2v: track 0.00 -> 194.8 mm, vias 0 -> 4
- net +3V3: track 0.00 -> 189.8 mm, vias 0 -> 8
- net +5V: track 0.00 -> 153.9 mm, vias 0 -> 3
- net /MT3608_1.2mHz_STEP-UP_CONVERTOR/power_input: track 0.00 -> 111.4 mm, vias 0 -> 2
- net +BATT: track 0.00 -> 103.7 mm, vias 0 -> 1
- net /DHT22_Data: track 0.00 -> 78.5 mm
- net /Motion_out: track 0.00 -> 67.1 mm, vias 0 -> 2
- net ESP_RX: track 0.00 -> 61.8 mm, vias 0 -> 3
- net /SIM808_GPRS_GPS_MODULE/LED_Netlight: track 0.00 -> 51.3 mm, vias 0 -> 1
- net /SIM808_GPRS_GPS_MODULE/SIM_VDD: track 0.00 -> 47.9 mm, vias 0 -> 1
- net /SIM808_GPRS_GPS_MODULE/SIM_RST: track 0.00 -> 45.6 mm, vias 0 -> 3
- net /SIM808_GPRS_GPS_MODULE/SIM_DATA: track 0.00 -> 41.1 mm, vias 0 -> 1
- net Net-(U10-FB): track 0.00 -> 37.7 mm
- net ESP_TX: track 0.00 -> 36.8 mm, vias 0 -> 2
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- added copper zone on B.Cu, net GND
- added copper zone on F.Cu, net GND
- added copper zone on In1.Cu, net GND
- added copper zone on In2.Cu, net GND
Other:
- board size 93.8 x 81.6 mm -> 77.8 x 81.6 mm
- copper layers 2 -> 4

Commit message: more Routing
Parts:
- added D3: SMLVN6RGB, LED_SMD:LED_ROHM_SMLVN6, F.Cu at (165.8, 52.3)
- added R16: 1k, Resistor_SMD:R_0402_1005Metric, F.Cu at (160.4, 50.3)
- added R17: 1k, Resistor_SMD:R_0402_1005Metric, F.Cu at (160.4, 52.3)
- added R18: 1k, Resistor_SMD:R_0402_1005Metric, F.Cu at (160.4, 54.2)
- added Switch+1: Switch+, TestPoint:TestPoint_Pad_D2.5mm, F.Cu at (173.2, 52.8)
- added Switch-1: Switch-, TestPoint:TestPoint_Pad_D2.5mm, F.Cu at (173.2, 59.1)
- moved U1 0.21 mm to (137.1, 55.2)
- renumbered TP31 to BAT+1, TP33 to BAT-1
Connections:
- U1 pad 18: unconnected-(U1-IO10-Pad18) -> /switch
- U1 pad 19: unconnected-(U1-IO11-Pad19) -> /blue
- U1 pad 20: unconnected-(U1-IO12-Pad20) -> /red
- U1 pad 21: unconnected-(U1-IO13-Pad21) -> /green
Routing:
- net /switch: track 0.00 -> 49.7 mm, vias 0 -> 2
- net /blue: track 0.00 -> 33.4 mm, vias 0 -> 2
- net /red: track 0.00 -> 30.8 mm, vias 0 -> 2
- net /green: track 0.00 -> 28.2 mm, vias 0 -> 2
- net GND: track 344.2 -> 362.4 mm, vias 232 -> 231
- net Net-(D3-GA): track 0.00 -> 3.77 mm
- net Net-(D3-BA): track 0.00 -> 3.76 mm
- net Net-(D3-RA): track 0.00 -> 3.38 mm
- net +3V3: track 189.8 -> 192.7 mm
- net /D+: track 31.9 -> 34.0 mm
- net /D-: track 32.7 -> 34.4 mm
- net Net-(Q1-B): track 2.13 -> 3.21 mm
- net ESP_TX: track 36.8 -> 37.7 mm
- net /MT3608_1.2mHz_STEP-UP_CONVERTOR/power_input: track 111.4 -> 110.5 mm
- net /SIM808_GPRS_GPS_MODULE/SIM7600_TXD: track 27.1 -> 26.6 mm

Commit message: more Routing
Parts:
- added +5V1: 5v, TestPoint:TestPoint_Loop_D2.50mm_Drill1.85mm, F.Cu at (172.7, 92.6)
- added GND1: GND, TestPoint:TestPoint_Loop_D2.50mm_Drill1.85mm, F.Cu at (172.7, 85.0)
- renumbered SW3 to BOOT1, SW2 to RESET1
Routing:
- net +5V: track 153.9 -> 205.3 mm, vias 3 -> 6
- net GND: track 362.4 -> 367.9 mm, vias 231 -> 234
- net /SIM808_GPRS_GPS_MODULE/LED_Status: track 33.1 -> 37.2 mm
- net /SIM808_GPRS_GPS_MODULE/SIM_DATA: track 41.1 -> 42.0 mm
Other:
- board text added: "Batt+"
- board text added: "Batt-"

Commit message: changinge mcu and shift level
Parts:
- removed C4: 10u, Capacitor_SMD:C_0402_1005Metric
- removed C5: 0.1u, Capacitor_SMD:C_0402_1005Metric
- removed Q2: BC817, Package_TO_SOT_SMD:SOT-23
- removed R99: 4.7k, Resistor_SMD:R_0402_1005Metric
- removed U1: ESP32-S3-WROOM-1, RF_Module:ESP32-S3-WROOM-1
- added C10: 10u, Capacitor_SMD:C_0402_1005Metric, F.Cu at (125.1, 51.1)
- added C11: 0.1u, Capacitor_SMD:C_0402_1005Metric, F.Cu at (124.0, 51.0)
- added C13: 22uF, Capacitor_SMD:C_0402_1005Metric, B.Cu at (113.8, 62.4)
- added C14: 100nF, Capacitor_SMD:C_0402_1005Metric, B.Cu at (112.8, 60.8)
- added C15: 22pF, Capacitor_SMD:C_0402_1005Metric, B.Cu at (109.7, 63.3)
- added C16: 22pF, Capacitor_SMD:C_0402_1005Metric, B.Cu at (106.8, 60.8)
- added C72: 100n, Capacitor_SMD:C_0402_1005Metric, F.Cu at (116.0, 90.0)
- added C73: 100n, Capacitor_SMD:C_0402_1005Metric, B.Cu at (115.2, 79.5)
- added C76: 100n, Capacitor_SMD:C_0402_1005Metric, F.Cu at (115.8, 85.9)
- added D10: B5819W, Diode_SMD:D_SOD-123, F.Cu at (115.5, 63.0)
- added D11: B5819W, Diode_SMD:D_SOD-123, B.Cu at (115.0, 66.2)
- added D12: B5819W, Diode_SMD:D_SOD-123, B.Cu at (121.1, 52.0)
- added D13: BAT54C, Package_TO_SOT_SMD:SOT-23, B.Cu at (125.0, 68.1)
- added IC1: RS0108YQ20, RS0108YQ20:SOP65P640X120-20N, B.Cu at (113.2, 84.9)
- added Q10: MMBT3904, Package_TO_SOT_SMD:SOT-23, B.Cu at (124.4, 56.1)
- added Q11: MMBT3904, Package_TO_SOT_SMD:SOT-23, B.Cu at (124.4, 61.1)
- added R100: 4.7k, Resistor_SMD:R_0402_1005Metric, F.Cu at (109.8, 87.0)
- added R101: 4.7k, Resistor_SMD:R_0402_1005Metric, F.Cu at (110.9, 89.6)
- added R11: 10k, Resistor_SMD:R_0402_1005Metric, B.Cu at (114.3, 60.8)
- added R110: 10k, Resistor_SMD:R_0402_1005Metric, B.Cu at (108.5, 87.8)
- added R111: 47k, Resistor_SMD:R_0402_1005Metric, F.Cu at (118.6, 87.8)
- added R112: 47k, Resistor_SMD:R_0402_1005Metric, B.Cu at (118.4, 81.9)
- added R19: 10k, Resistor_SMD:R_0402_1005Metric, F.Cu at (112.9, 65.2)
- added R20: 10k, Resistor_SMD:R_0402_1005Metric, B.Cu at (120.8, 56.3)
- added R21: 10k, Resistor_SMD:R_0402_1005Metric, B.Cu at (123.3, 58.8)
- added R22: 220R, Resistor_SMD:R_0402_1005Metric, B.Cu at (124.0, 64.6)
- added U6: ESP32-WROOM-32, RF_Module:ESP32-WROOM-32, F.Cu at (137.4, 58.1)
- added U8: CH340T(SSOP20W), Package_SO:SSOP-20_5.3x7.2mm_P0.65mm, B.Cu at (112.5, 54.4)
- added Y1: 12MHz, Crystal:Crystal_SMD_2520-4Pin_2.5x2.0mm, B.Cu at (109.5, 61.0)
- moved Q1 11.5 mm to (112.5, 86.6), turned to 90 degrees
- moved C71 5.58 mm to (108.7, 91.2), turned to 180 degrees
- moved R82 0.43 mm to (108.5, 89.7), turned to 180 degrees
Connections:
- IC4 pad 3: GND -> /SIM808_GPRS_GPS_MODULE/pwrkey
- IC4 pad 54: unconnected-(IC4-FLIGHTMODE-Pad54) -> /SIM808_GPRS_GPS_MODULE/Flight
- IC4 pad 69: unconnected-(IC4-RI-Pad69) -> /SIM808_GPRS_GPS_MODULE/RI
- Q1 pad 2: /SIM808_GPRS_GPS_MODULE/SIM7600_TXD -> /SIM808_GPRS_GPS_MODULE/pwrkey
- Q1 pad 3: ESP_RX -> GND
Routing:
- net /D-: track 34.4 -> 9.35 mm
- net /D+: track 34.0 -> 9.35 mm
- net /SIM808_GPRS_GPS_MODULE/SIM7600_RXD: track 36.5 -> 14.0 mm
- net +3V3: track 192.9 -> 171.3 mm
- net /SIM808_GPRS_GPS_MODULE/SIM7600_TXD: track 26.6 -> 9.20 mm
- net ESP_RX: track 61.8 -> 51.5 mm, vias 3 -> 2
- net /DHT22_Data: track 78.5 -> 70.5 mm
- net GND: track 367.9 -> 360.3 mm
- net /~{esp_rst}: track 16.7 -> 9.29 mm, vias 2 -> 1
- net /SIM808_GPRS_GPS_MODULE/1.8v_OUT: track 27.9 -> 21.1 mm
- net ESP_TX: track 37.7 -> 31.8 mm, vias 2 -> 0
- net /boot: track 10.0 -> 4.29 mm
- net /Motion_out: track 66.9 -> 63.8 mm, vias 2 -> 1
- net /blue: track 33.4 -> 30.5 mm
- net /switch: track 49.7 -> 46.7 mm
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