File: schematic/schematic.kicad_pcb (KiCad board)
At the start: 4 copper layers, 77.8 x 81.6 mm, 152 parts, among them IC1 RS0108YQ20, IC2 AS312, IC3 TPS630250RNCR, IC4 SIM7600G-H_R2, J1 SIM7155-6-1-14-A, J3 USB_C_Receptacle_USB2.0, Q1 BC817, Q10 MMBT3904, Q11 MMBT3904, Q15 SI2302, Q16 SI2302, Q8 NCE6005AR, Q9 NCE6005AR, U10 TPS56339DDC, U2 MT3608, U3 AM2302, U4 TP4056, U6 ESP32-WROOM-32, U8 CH340T(SSOP20W), Y1 12MHz

Commit message: Ground and power routing...
Parts:
- added C1: 22u, Capacitor_SMD:C_0402_1005Metric, B.Cu at (178.7, 67.9)
- added C1: 22u, Capacitor_SMD:C_0402_1005Metric, B.Cu at (178.4, 74.2)
- added C1: 22u, Capacitor_SMD:C_0402_1005Metric, B.Cu at (182.6, 58.6)
- added C2: 22u, Capacitor_SMD:C_0402_1005Metric, B.Cu at (179.5, 71.9)
- added C2: 22u, Capacitor_SMD:C_0402_1005Metric, B.Cu at (183.6, 56.2)
- added C2: 22u, Capacitor_SMD:C_0402_1005Metric, B.Cu at (179.8, 65.6)
- added C3: 100n, Capacitor_SMD:C_0402_1005Metric, B.Cu at (185.1, 56.3)
- added C3: 100n, Capacitor_SMD:C_0402_1005Metric, B.Cu at (181.2, 65.6)
- added C3: 100n, Capacitor_SMD:C_0402_1005Metric, B.Cu at (180.9, 71.9)
- added C7: 100n, Capacitor_SMD:C_0402_1005Metric, B.Cu at (167.8, 60.2)
- added C7: 100n, Capacitor_SMD:C_0402_1005Metric, B.Cu at (171.7, 50.8)
- added C7: 100n, Capacitor_SMD:C_0402_1005Metric, B.Cu at (167.5, 66.4)
- added C8: 22u, Capacitor_SMD:C_0402_1005Metric, B.Cu at (173.2, 50.8)
- added C8: 22u, Capacitor_SMD:C_0402_1005Metric, B.Cu at (169.4, 60.2)
- added C8: 22u, Capacitor_SMD:C_0402_1005Metric, B.Cu at (169.1, 66.4)
- added C9: 22u, Capacitor_SMD:C_0402_1005Metric, B.Cu at (174.7, 50.8)
- added C9: 22u, Capacitor_SMD:C_0402_1005Metric, B.Cu at (170.8, 60.2)
- added C9: 22u, Capacitor_SMD:C_0402_1005Metric, B.Cu at (170.5, 66.4)
- added D1: SS54, Diode_SMD:D_SMA, B.Cu at (168.7, 71.3)
- added D1: SS54, Diode_SMD:D_SMA, B.Cu at (172.8, 55.7)
- added D1: SS54, Diode_SMD:D_SMA, B.Cu at (169.0, 65.1)
- added L1: 22uH, Inductor_SMD:L_Chilisin_BMRG00101030, B.Cu at (173.7, 80.4)
- added L1: 22uH, Inductor_SMD:L_Chilisin_BMRG00101030, B.Cu at (177.8, 64.8)
- added L1: 22uH, Inductor_SMD:L_Chilisin_BMRG00101030, B.Cu at (174.0, 74.2)
- added R1: 10K, Resistor_SMD:R_0402_1005Metric, B.Cu at (177.9, 71.9)
- added R1: 10K, Resistor_SMD:R_0402_1005Metric, B.Cu at (178.2, 65.6)
- added R1: 10K, Resistor_SMD:R_0402_1005Metric, B.Cu at (182.0, 56.3)
- added R2: 120K, Resistor_SMD:R_0402_1005Metric, B.Cu at (176.6, 53.0)
- added R2: 120K, Resistor_SMD:R_0402_1005Metric, B.Cu at (172.8, 62.3)
- added R2: 120K, Resistor_SMD:R_0402_1005Metric, B.Cu at (172.5, 68.6)
- added R3: 16K, Resistor_SMD:R_0402_1005Metric, B.Cu at (173.2, 60.5)
- added R3: 16K, Resistor_SMD:R_0402_1005Metric, B.Cu at (177.1, 51.2)
- added R3: 16K, Resistor_SMD:R_0402_1005Metric, B.Cu at (172.9, 66.8)
- added U2: MT3608, Package_TO_SOT_SMD:SOT-23-6, B.Cu at (174.5, 72.7)
- added U2: MT3608, Package_TO_SOT_SMD:SOT-23-6, B.Cu at (174.8, 66.5)
- added U2: MT3608, Package_TO_SOT_SMD:SOT-23-6, B.Cu at (178.6, 57.1)
