File: schematic/BUCK_CONVERTER_3V3_2A_TPS56339DDCR.kicad_sch (KiCad schematic)
At the start: 14 parts, among them U10 TPS56339DDC

Commit message: Routing
Parts:
- L5: footprint greencharge-footprints:YSPI0530-XXX -> Inductor_SMD:L_Chilisin_BMRx00050512-B; MPN YSPI0530-4R7M -> YSPI0530S-4R7M
Changed lines of the file:
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@@
 			)
 		)
-		(property "Footprint" "greencharge-footprints:YSPI0530-XXX"
+		(property "Footprint" "Inductor_SMD:L_Chilisin_BMRx00050512-B"
 			(at 191.77 46.99 0)
 			(effects
@@
 			)
 		)
-		(property "MPN" "YSPI0530-4R7M"
+		(property "MPN" "YSPI0530S-4R7M"
 			(at 194.31 49.53 0)
 			(effects
