File: schematic/LIPO_BAT_CHARGER_TP4056.kicad_sch (KiCad schematic)
At the start: 22 parts, among them J9 BATT_CONNECTOR, U4 TP4056

Commit message: Routing
Parts:
- removed TH1: 10K, Resistor_SMD:R_0402_1005Metric, symbol Device:Thermistor_NTC
- J9: footprint MACHADA_footprints:2pin_2mm_jst_v_bat_S2B-PH-SM4-TB -> TerminalBlock_Phoenix:TerminalBlock_Phoenix_PTSM-0,5-2-HV-2.5-SMD_1x02-1MP_P2.50mm_Vertical
- U4: footprint MACHADA_footprints:SOP127P600X175-9N -> tp4056:SOIC127P600X175-9N
Changed lines of the file:
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@@
-	)
-	(junction
-		(at 204.47 111.76)
-		(diameter 0)
-		(color 0 0 0 0)
 	)
 	(junction
@@
 	)
 	(junction
-		(at 204.47 100.33)
-		(diameter 0)
-		(color 0 0 0 0)
-	)
-	(junction
 		(at 95.25 55.88)
 		(diameter 0)
@@
 	(wire
 		(pts
-			(xy 204.47 109.22) (xy 204.47 111.76)
-		)
-		(stroke
-			(width 0)
-			(type default)
-		)
-	)
-	(wire
-		(pts
 			(xy 184.15 58.42) (xy 194.31 58.42)
 		)
@@
 		(pts
 			(xy 227.33 58.42) (xy 274.32 58.42)
-		)
-		(stroke
-			(width 0)
-			(type default)
-		)
-	)
-	(wire
-		(pts
-			(xy 204.47 100.33) (xy 204.47 101.6)
 		)
 		(stroke
@@
 			)
 		)
-		(property "Footprint" "MACHADA_footprints:2pin_2mm_jst_v_bat_S2B-PH-SM4-TB"
+		(property "Footprint" "TerminalBlock_Phoenix:TerminalBlock_Phoenix_PTSM-0,5-2-HV-2.5-SMD_1x02-1MP_P2.50mm_Vertical"
 			(at 241.3 81.28 0)
 			(effects
@@
 	)
 	(symbol
-		(lib_id "Device:Thermistor_NTC")
-		(at 204.47 105.41 0)
-		(unit 1)
-		(exclude_from_sim no)
-		(in_bom yes)
-		(on_board no)
-		(dnp no)
-		(fields_autoplaced yes)
-		(property "Reference" "TH1"
-			(at 207.01 104.4575 0)
-			(effects
-				(font
-					(size 1.27 1.27)
-				)
-				(justify left)
-			)
-		)
-		(property "Value" "10K"
-			(at 207.01 106.9975 0)
-			(effects
-				(font
-					(size 1.27 1.27)
-				)
-				(justify left)
-			)
-		)
-		(property "Footprint" "Resistor_SMD:R_0402_1005Metric"
-			(at 204.47 104.14 0)
-			(effects
-				(font
-					(size 1.27 1.27)
-				)
-				(hide yes)
-			)
-		)
-		(property "Datasheet" "~"
-			(at 204.47 104.14 0)
-			(effects
-				(font
-					(size 1.27 1.27)
-				)
-				(hide yes)
-			)
-		)
-		(property "Description" ""
-			(at 204.47 105.41 0)
-			(effects
-				(font
-					(size 1.27 1.27)
-				)
-				(hide yes)
-			)
-		)
-		(pin "1"
-		)
-		(pin "2"
-		)
-		(instances
-			(project "schematic"
-				(path "/374f5031-bd65-4a4b-92ce-befdd0c9f08b/91cef089-9175-4786-91ce-da26d26da4e3"
-					(reference "TH1")
-					(unit 1)
-				)
-			)
-		)
-	)
-	(symbol
 		(lib_id "Device:C_Small")
 		(at 85.09 60.96 0)
@@
 			)
 		)
-		(property "Footprint" "MACHADA_footprints:SOP127P600X175-9N"
+		(property "Footprint" "tp4056:SOIC127P600X175-9N"
 			(at 171.45 73.66 0)
 			(effects

Commit message: more Routing
Parts:
- renumbered TP31 to BAT+1, TP33 to BAT-1
Changed lines of the file:
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@@
 		(on_board yes)
 		(dnp no)
-		(property "Reference" "TP31"
+		(property "Reference" "BAT+1"
 			(at 264.16 71.628 0)
 			(effects
@@
 			(project "schematic"
 				(path "/374f5031-bd65-4a4b-92ce-befdd0c9f08b/91cef089-9175-4786-91ce-da26d26da4e3"
-					(reference "TP31")
+					(reference "BAT+1")
 					(unit 1)
 				)
@@
 		(on_board yes)
 		(dnp no)
-		(property "Reference" "TP33"
+		(property "Reference" "BAT-1"
 			(at 267.97 81.788 0)
 			(effects
@@
 			(project "schematic"
 				(path "/374f5031-bd65-4a4b-92ce-befdd0c9f08b/91cef089-9175-4786-91ce-da26d26da4e3"
-					(reference "TP33")
+					(reference "BAT-1")
 					(unit 1)
 				)

Commit message: changinge mcu and shift level
Parts:
- removed J9: BATT_CONNECTOR, TerminalBlock_Phoenix:TerminalBlock_Phoenix_PTSM-0,5-2-HV-2.5-SMD_1x02-1MP_P2.50mm_Vertical, symbol Connector_Generic:Conn_01x02
Changed lines of the file:
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@@
-	)
-	(junction
-		(at 236.22 76.835)
-		(diameter 0)
-		(color 0 0 0 0)
 	)
 	(junction
@@
 	)
 	(junction
-		(at 265.43 86.36)
-		(diameter 0)
-		(color 0 0 0 0)
-	)
-	(junction
 		(at 227.33 58.42)
 		(diameter 0)
@@
 	(wire
 		(pts
-			(xy 236.22 86.36) (xy 265.43 86.36)
-		)
-		(stroke
-			(width 0)
-			(type default)
-		)
-	)
-	(wire
-		(pts
 			(xy 186.69 100.33) (xy 204.47 100.33)
 		)
@@
 	(wire
 		(pts
-			(xy 236.22 83.82) (xy 236.22 86.36)
-		)
-		(stroke
-			(width 0)
-			(type default)
-		)
-	)
-	(wire
-		(pts
-			(xy 227.33 76.835) (xy 236.22 76.835)
-		)
-		(stroke
-			(width 0)
-			(type default)
-		)
-	)
-	(wire
-		(pts
 			(xy 143.51 63.5) (xy 148.59 63.5)
 		)
@@
 	(wire
 		(pts
-			(xy 236.22 76.835) (xy 236.22 81.28)
-		)
-		(stroke
-			(width 0)
-			(type default)
-		)
-	)
-	(wire
-		(pts
-			(xy 251.46 76.835) (xy 236.22 76.835)
+			(xy 227.33 76.835) (xy 251.46 76.835)
 		)
 		(stroke
@@
 					(unit 1)
 				)
-			)
-		)
-	)
-	(symbol
-		(lib_id "Connector_Generic:Conn_01x02")
-		(at 241.3 81.28 0)
-		(unit 1)
-		(exclude_from_sim no)
-		(in_bom yes)
-		(on_board yes)
-		(dnp no)
-		(property "Reference" "J9"
-			(at 241.3 72.39 0)
-			(effects
-				(font
-					(size 1.27 1.27)
-				)
-			)
-		)
-		(property "Value" "BATT_CONNECTOR"
-			(at 239.395 74.93 0)
-			(effects
-				(font
-					(size 1.27 1.27)
-				)
-			)
-		)
-		(property "Footprint" "TerminalBlock_Phoenix:TerminalBlock_Phoenix_PTSM-0,5-2-HV-2.5-SMD_1x02-1MP_P2.50mm_Vertical"
-			(at 241.3 81.28 0)
-			(effects
-				(font
-					(size 1.27 1.27)
-				)
-				(hide yes)
-			)
-		)
-		(property "Datasheet" "~"
-			(at 241.3 81.28 0)
-			(effects
-				(font
-					(size 1.27 1.27)
-				)
-				(hide yes)
-			)
-		)
-		(property "Description" ""
-			(at 241.3 81.28 0)
-			(effects
-				(font
-					(size 1.27 1.27)
-				)
-				(hide yes)
-			)
-		)
-		(pin "1"
-		)
-		(pin "2"
-		)
-		(instances
-			(project "schematic"
-				(path "/374f5031-bd65-4a4b-92ce-befdd0c9f08b/91cef089-9175-4786-91ce-da26d26da4e3"
-					(reference "J9")
-					(unit 1)
-				)
